File: Tube_Audio/Helper_Circuits/EFB_Bias_Supply/EFB_Bias_Supply.kicad_pcb (KiCad board)
At the start: 2 copper layers, 59.7 x 41.9 mm, 20 parts, among them J1 Screw_Terminal_01x02, J2 Screw_Terminal_01x03, J3 Screw_Terminal_01x02, Q1 KSA1013, Q2 KSA1013

Commit message: Clarify trademark status in all materials.
Other:
- board text added: "D Gillespie Designs EFB(tm) Bias Supply, board rev. 1"
- board text removed: "Gillespie EFB(tm) Bias Supply, board rev. 1"
Changed lines of the file:
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@@
     (links 26)
     (no_connects 0)
-    (area 91.364999 69.774999 151.205001 111.835001)
+    (area 78.510001 62.07 164.06 119.540001)
     (thickness 1.6)
     (drawings 15)
@@
     (effects (font (size 1 1) (thickness 0.25)))
   )
-  (gr_text "Gillespie EFB(tm)\nBias Supply, board rev. 1" (at 148.59 91.44 90) (layer F.SilkS)
+  (gr_text "D Gillespie Designs EFB(tm)\nBias Supply, board rev. 1" (at 148.59 91.44 90) (layer F.SilkS)
     (effects (font (size 1 1) (thickness 0.25)))
   )
