File: Tube_Audio/Helper_Circuits/EFB_Bias_Supply/EFB_Bias_Supply.sch (KiCad schematic (older format))
At the start: 16 parts, among them J1 Screw_Terminal_01x02, J2 Screw_Terminal_01x03, J3 Screw_Terminal_01x02, Q1 KSA1013, Q2 KSA1013

Commit message: Clarify trademark status in all materials.
Other:
- note added: "EFB(tm) and Enhanced Fixed Bias(tm) are trademarks of\nD Gillespie Designs and are used with permission.\n\nCircuit is copyright D Gillespie Designs, and is used with permission."
Changed lines of the file:
@@
 Wire Wire Line
 	8250 3750 8250 3650
+Text Notes 5400 5800 0    60   ~ 0
+EFB(tm) and Enhanced Fixed Bias(tm) are trademarks of\nD Gillespie Designs and are used with permission.\n\nCircuit is copyright D Gillespie Designs, and is used with permission.
 $EndSCHEMATC
