File: Tube_Audio/Helper_Circuits/EFB_Cathode_Regulator/EFB_Cathode_Regulator.kicad_pcb (KiCad board)
At the start: 2 copper layers, 38.1 x 24.9 mm, 9 parts, among them J1 Screw_Terminal_01x03, J2 Screw_Terminal_01x02, U1 LM337

Commit message: Clarify trademark status in all materials.
Other:
- board text added: "EFB(tm) Cathode Regulator Circuit by D Gillepsie Designs"
- board text removed: "EFB(tm) Cathode Regulator Circuit by David Gillespie."
- board text removed: "www.sfelectronworks.com"
Changed lines of the file:
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@@
     (area 136.318 72.829 186.92 105.823828)
     (thickness 1.6)
-    (drawings 13)
+    (drawings 12)
     (tracks 44)
     (zones 0)
@@
     (visible_elements FFFFFF7F)
     (pcbplotparams
-      (layerselection 0x010f0_80000001)
+      (layerselection 0x210f0_80000001)
       (usegerberextensions false)
       (excludeedgelayer true)
@@
     )
   )
-  (gr_text www.sfelectronworks.com (at 155.448 92.71) (layer B.SilkS)
-    (effects (font (size 0.75 0.75) (thickness 0.1875)) (justify mirror))
-  )
   (gr_text "Board (c) 2018 Jason R. Thorpe." (at 154.94 87.376) (layer B.SilkS)
     (effects (font (size 0.75 0.75) (thickness 0.1875)) (justify mirror))
   )
-  (gr_text "EFB(tm) Cathode Regulator\nCircuit by David Gillespie." (at 154.686 81.788) (layer B.SilkS)
+  (gr_text "EFB(tm) Cathode Regulator\nCircuit by D Gillepsie Designs" (at 154.686 81.788) (layer B.SilkS)
     (effects (font (size 0.75 0.75) (thickness 0.1875)) (justify mirror))
   )
@@
     (effects (font (size 1.5 1.5) (thickness 0.3)))
   )
-  (segment (start 169.926 79.756) (end 167.64 79.756) (width 1) (layer B.Cu) (net 1) (status 400000))
-  (segment (start 151.13 80.01) (end 151.13 77.724) (width 1) (layer B.Cu) (net 1) (status 800000))
+  (segment (start 169.926 79.756) (end 167.64 79.756) (width 1) (layer B.Cu) (net 1))
+  (segment (start 151.13 80.01) (end 151.13 77.724) (width 1) (layer B.Cu) (net 1))
   (segment (start 153.416 82.296) (end 151.13 80.01) (width 1) (layer B.Cu) (net 1))
   (segment (start 165.1 82.296) (end 153.416 82.296) (width 1) (layer B.Cu) (net 1))
   (segment (start 167.64 79.756) (end 165.1 82.296) (width 1) (layer B.Cu) (net 1))
-  (segment (start 167.092 95.798) (end 169.632 95.798) (width 1) (layer B.Cu) (net 1) (status 400000))
-  (segment (start 171.958 81.788) (end 169.926 79.756) (width 1) (layer B.Cu) (net 1) (status 800000))
+  (segment (start 167.092 95.798) (end 169.632 95.798) (width 1) (layer B.Cu) (net 1))
+  (segment (start 171.958 81.788) (end 169.926 79.756) (width 1) (layer B.Cu) (net 1))
   (segment (start 171.958 93.472) (end 171.958 81.788) (width 1) (layer B.Cu) (net 1))
   (segment (start 169.632 95.798) (end 171.958 93.472) (width 1) (layer B.Cu) (net 1))
-  (segment (start 169.926 77.756) (end 165.536 77.756) (width 1) (layer F.Cu) (net 2) (status 400000))
-  (segment (start 165.536 77.756) (end 164.552 78.74) (width 1) (layer F.Cu) (net 2) (status 800000))
+  (segment (start 169.926 77.756) (end 165.536 77.756) (width 1) (layer F.Cu) (net 2))
+  (segment (start 165.536 77.756) (end 164.552 78.74) (width 1) (layer F.Cu) (net 2))
   (segment (start 164.552 78.74) (end 164.552 80.558) (width 1) (layer B.Cu) (net 2))
   (segment (start 153.67 79.248) (end 153.67 77.724) (width 1) (layer B.Cu) (net 2))
