File: Tube_Audio/6AS7_Pre_amp_Mk_I/STPre6080PSU.kicad_pcb (KiCad board)
At the start: 2 copper layers, 94 x 82.5 mm, 26 parts, among them J301 Screw_Terminal_01x02, J302 Screw_Terminal_01x02, J303 Screw_Terminal_01x02, J304 Screw_Terminal_01x03

Commit message: Checkpoint -- getting closer to laying out the tone control PCB.
Changed lines of the file:
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@@
       (effects (font (size 1 1) (thickness 0.15)))
     )
-    (fp_text value MountingHole_3.5mm_Pad (at 0 4.5) (layer F.Fab)
+    (fp_text value MountingHole_3.5mm_Pad (at 0 4.5) (layer F.Fab) hide
       (effects (font (size 1 1) (thickness 0.15)))
     )
@@
       (effects (font (size 1 1) (thickness 0.15)))
     )
-    (fp_text value MountingHole_3.5mm_Pad (at 0 4.5) (layer F.Fab)
+    (fp_text value MountingHole_3.5mm_Pad (at 0 4.5) (layer F.Fab) hide
       (effects (font (size 1 1) (thickness 0.15)))
     )
@@
       (effects (font (size 1 1) (thickness 0.15)))
     )
-    (fp_text value 270uF (at 3.75 10.25) (layer F.Fab)
+    (fp_text value 270uF (at 3.75 10.25) (layer F.SilkS)
       (effects (font (size 1 1) (thickness 0.15)))
     )
@@
       (effects (font (size 1 1) (thickness 0.15)))
     )
-    (fp_text value 270uF (at 3.75 10.25) (layer F.Fab)
+    (fp_text value 270uF (at 3.75 10.25) (layer F.SilkS)
       (effects (font (size 1 1) (thickness 0.15)))
     )
@@
       (effects (font (size 1 1) (thickness 0.15)))
     )
-    (fp_text value 270uF (at 3.75 10.25) (layer F.Fab)
+    (fp_text value 270uF (at 3.75 10.25) (layer F.SilkS)
       (effects (font (size 1 1) (thickness 0.15)))
     )
@@
       (effects (font (size 1 1) (thickness 0.15)))
     )
-    (fp_text value 47uF (at 2.5 7.5 90) (layer F.Fab)
+    (fp_text value 47uF (at 2.5 7.5 90) (layer F.SilkS)
       (effects (font (size 1 1) (thickness 0.15)))
     )
@@
       (effects (font (size 1 1) (thickness 0.15)))
     )
-    (fp_text value 270uF (at 3.75 10.25 90) (layer F.Fab)
+    (fp_text value 270uF (at 3.75 10.25 90) (layer F.SilkS)
       (effects (font (size 1 1) (thickness 0.15)))
     )
@@
       (effects (font (size 1 1) (thickness 0.15)))
     )
-    (fp_text value 100uF (at 3.75 10.25) (layer F.Fab)
+    (fp_text value 100uF (at 3.75 10.25) (layer F.SilkS)
       (effects (font (size 1 1) (thickness 0.15)))
     )
@@
       (effects (font (size 1 1) (thickness 0.15)))
     )
-    (fp_text value 820uF (at 5 13.75) (layer F.Fab)
+    (fp_text value 820uF (at 5 13.75) (layer F.SilkS)
       (effects (font (size 1 1) (thickness 0.15)))
     )
@@
       (effects (font (size 1 1) (thickness 0.15)))
     )
-    (fp_text value 820uF (at 5 13.75) (layer F.Fab)
+    (fp_text value 820uF (at 5 13.75) (layer F.SilkS)
       (effects (font (size 1 1) (thickness 0.15)))
     )
@@
       (effects (font (size 1 1) (thickness 0.15)))
     )
-    (fp_text value 1N4007 (at 5.08 2.47) (layer F.Fab)
+    (fp_text value 1N4007 (at 5.08 2.47) (layer F.SilkS)
       (effects (font (size 1 1) (thickness 0.15)))
     )
@@
       (effects (font (size 1 1) (thickness 0.15)))
     )
-    (fp_text value 1N4007 (at 5.08 2.47) (layer F.Fab)
+    (fp_text value 1N4007 (at 5.08 2.47) (layer F.SilkS)
       (effects (font (size 1 1) (thickness 0.15)))
     )
@@
       (effects (font (size 1 1) (thickness 0.15)))
     )
-    (fp_text value 22K (at 3.81 2.37) (layer F.Fab)
+    (fp_text value 22K (at 3.81 2.37) (layer F.SilkS)
       (effects (font (size 1 1) (thickness 0.15)))
     )
@@
       (effects (font (size 1 1) (thickness 0.15)))
     )
-    (fp_text value 12K (at 3.81 2.37) (layer F.Fab)
+    (fp_text value 12K (at 3.81 2.37) (layer F.SilkS)
       (effects (font (size 1 1) (thickness 0.15)))
     )
@@
       (effects (font (size 1 1) (thickness 0.15)))
     )
-    (fp_text value 2.2K (at 3.81 2.37) (layer F.Fab)
+    (fp_text value 2.2K (at 3.81 2.37) (layer F.SilkS)
       (effects (font (size 1 1) (thickness 0.15)))
     )
@@
       (effects (font (size 1 1) (thickness 0.15)))
     )
-    (fp_text value 3.9K (at 3.81 2.37) (layer F.Fab)
+    (fp_text value 3.9K (at 3.81 2.37) (layer F.SilkS)
       (effects (font (size 1 1) (thickness 0.15)))
     )
@@
       (effects (font (size 1 1) (thickness 0.15)))
     )
-    (fp_text value 500R (at 0 2.52) (layer F.Fab)
+    (fp_text value 500R (at 0 2.52) (layer F.SilkS)
       (effects (font (size 1 1) (thickness 0.15)))
     )
