File: Tube_Audio/6AS7_Pre_amp_Mk_I/STPre6080PSU.kicad_pcb (KiCad board)
At the start: 2 copper layers, 94 x 82.5 mm, 26 parts, among them J301 Screw_Terminal_01x02, J302 Screw_Terminal_01x02, J303 Screw_Terminal_01x02, J304 Screw_Terminal_01x03

Commit message: Add high voltage warnings.
Parts:
- added REF**: Symbol_HighVoltage_Type2_FSilk_VerySmall, jrt-Graphics:Symbol_HighVoltage_Type2_FSilk_VerySmall, F.Cu at (167.6, 106.7)
Other:
- board text added: "HIGH VOLTAGE!"
Changed lines of the file:
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@@
   (general
     (thickness 1.6)
-    (drawings 22)
+    (drawings 23)
     (tracks 82)
     (zones 0)
-    (modules 26)
+    (modules 27)
     (nets 12)
   )
@@
     (add_net "Net-(C307-Pad1)")
   )
+  (module jrt-Graphics:Symbol_HighVoltage_Type2_FSilk_VerySmall (layer F.Cu)
+    (at 167.64 106.68)
+    (descr "Symbol, High Voltage, Type 2, FSilk, Very Small,")
+    (tags "Symbol, High Voltage, Type 2, FSilk, Very Small,")
+    (attr virtual)
+    (fp_text reference REF** (at -0.127 -5.715) (layer F.SilkS) hide
+      (effects (font (size 1 1) (thickness 0.15)))
+    )
+    (fp_text value Symbol_HighVoltage_Type2_FSilk_VerySmall (at -0.381 4.572) (layer F.Fab) hide
+      (effects (font (size 1 1) (thickness 0.15)))
+    )
+    (fp_line (start -4.699 2.794) (end 0 -4.191) (layer F.SilkS) (width 0.381))
+    (fp_line (start 4.699 2.794) (end -4.699 2.794) (layer F.SilkS) (width 0.381))
+    (fp_line (start 0 -4.191) (end 4.699 2.794) (layer F.SilkS) (width 0.381))
+    (fp_line (start -0.49784 2.19964) (end -0.59944 1.30048) (layer F.SilkS) (width 0.381))
+    (fp_line (start 0.29972 -0.59944) (end -0.49784 2.19964) (layer F.SilkS) (width 0.381))
+    (fp_line (start -0.89916 0.20066) (end 0.29972 -0.59944) (layer F.SilkS) (width 0.381))
+    (fp_line (start -0.09906 -2.79908) (end -0.89916 0.20066) (layer F.SilkS) (width 0.381))
+    (fp_line (start -0.49784 2.19964) (end 0.1016 1.50114) (layer F.SilkS) (width 0.381))
+    (fp_line (start -0.89916 0.20066) (end 0.40132 -2.60096) (layer F.SilkS) (width 0.381))
+    (fp_line (start 0.70104 -0.89916) (end 0.1016 -0.50038) (layer F.SilkS) (width 0.381))
+    (fp_line (start -0.49784 2.19964) (end 0.70104 -0.89916) (layer F.SilkS) (width 0.381))
+  )
   (module TestPoint:TestPoint_2Pads_Pitch2.54mm_Drill0.8mm (layer F.Cu)
     (at 119.38 85.09 270)
@@
     )
   )
+  (gr_text "HIGH\nVOLTAGE!" (at 168.91 129.54) (layer F.SilkS)
+    (effects (font (size 1.5 1.5) (thickness 0.3) italic))
+  )
   (dimension 83.82 (width 0.15) (layer Dwgs.User)
