File: Tube_Audio/6AS7_Pre_amp_Mk_I/STPre6080.sch (KiCad schematic (older format))
At the start: 27 parts, among them SW1 SW_Rotary2x4_CandK_A20403RNZQ, SW2 SW_DPDT_x2, U1 ECC83, U2 2ChanCCSLoad, U3 6AS7

Commit message: Checkpoint -- getting closer to laying out the tone control PCB.
Parts:
- R4, R8: value 1.2K -> 1.8K
Connections:
- net +300V renamed +250V
Other:
- note added: "Power Supply\n(PCB)"
- note removed: "Power Supply"
Changed lines of the file:
@@
 L_output
 $Comp
-L jrt-Power:+300V #PWR?
+L jrt-Power:+250V #PWR?
 U 1 1 5D97E177
 P 7000 1000
@@
 AR Path="/5DA0A318/5D97E177" Ref="#PWR?"  Part="1"
 F 0 "#PWR?" H 7000 850 50  0001 C CNN
-F 1 "+300V" H 7015 1173 50  0000 C CNN
+F 1 "+250V" H 7015 1173 50  0000 C CNN
 F 2 "" H 7000 1000 50  0001 C CNN
 F 3 "" H 7000 1000 50  0001 C CNN
@@
 AR Path="/5DA0A318/5D97E19B" Ref="R?"  Part="1"
 F 0 "R4" H 6959 2546 50  0000 L CNN
-F 1 "1.2K" H 6959 2455 50  0000 L CNN
+F 1 "1.8K" H 6959 2455 50  0000 L CNN
 F 2 "" H 6900 2500 50  0001 C CNN
 F 3 "~" H 6900 2500 50  0001 C CNN
@@
 	6400 2650 6900 2650
 $Comp
-L jrt-Power:+300V #PWR?
+L jrt-Power:+250V #PWR?
 U 1 1 5DAA7C62
 P 9150 1000
@@
 AR Path="/5DA0A318/5DAA7C62" Ref="#PWR?"  Part="1"
 F 0 "#PWR?" H 9150 850 50  0001 C CNN
-F 1 "+300V" H 9165 1173 50  0000 C CNN
+F 1 "+250V" H 9165 1173 50  0000 C CNN
 F 2 "" H 9150 1000 50  0001 C CNN
 F 3 "" H 9150 1000 50  0001 C CNN
@@
 AR Path="/5DA0A318/5DAA7C80" Ref="R?"  Part="1"
 F 0 "R8" H 9109 2546 50  0000 L CNN
-F 1 "1.2K" H 9109 2455 50  0000 L CNN
+F 1 "1.8K" H 9109 2455 50  0000 L CNN
 F 2 "" H 9050 2500 50  0001 C CNN
 F 3 "~" H 9050 2500 50  0001 C CNN
@@
 $EndSheet
 Text Notes 2650 6850 0    50   Italic 10
-Power Supply
+Power Supply\n(PCB)
 $EndSCHEMATC

Commit message: Removed the heater circuit sheet -- that has been spun off into a separate project.
Other:
- note added: "(Separate PCB)"
- note removed: "Heater configuration circuit"
Changed lines of the file:
@@
 Wire Wire Line
 	7050 4800 7150 4800
-$Sheet
-S 4400 6150 1700 1300
-U 5DC527CD
-F0 "STPre6080Heaters" 50
-F1 "STPre6080Heaters.sch" 50
-$EndSheet
-Text Notes 4750 7300 0    50   Italic 10
-Heater configuration circuit
 Wire Notes Line
 	5350 700  10300 700
@@
 Text Notes 2650 6850 0    50   Italic 10
 Power Supply\n(PCB)
+Text Notes 6200 3800 0    50   ~ 0
+(Separate PCB)
 $EndSCHEMATC

Commit message: Rename 2ChamCCSLoad to CCS_Load_x2
Parts:
- U2: value 2ChanCCSLoad -> CCS_Load_x2; symbol jrt-Regulators:2ChanCCSLoad -> jrt-Regulators:CCS_Load_x2
Changed lines of the file:
@@
 $Descr USLetter 11000 8500
 encoding utf-8
-Sheet 1 4
+Sheet 1 3
 Title "6AS7 Pre-amp Mk I"
 Date "2019-09-19"
@@
 100V
 $Comp
-L jrt-Regulators:2ChanCCSLoad U2
+L jrt-Regulators:CCS_Load_x2 U2
 U 1 1 5DB45136
 P 5900 3600
 F 0 "U2" H 6228 3646 50  0000 L CNN
-F 1 "2ChanCCSLoad" H 6228 3555 50  0000 L CNN
+F 1 "CCS_Load_x2" H 6228 3555 50  0000 L CNN
 F 2 "" H 5900 3600 50  0001 C CNN
 F 3 "" H 5900 3600 50  0001 C CNN
