File: Misc_Audio/RAdLib/Clock_Source.sch (KiCad schematic (older format))
At the start: 5 parts, among them U101 74AHCT04, Y101 3.58MHz Crystal

Commit message: Checkpoint ... board is close to being done.  Still need to tweak the ground plane.
Parts:
- added C101: .1uF, Capacitor_THT:C_Disc_D5.0mm_W2.5mm_P2.50mm, symbol Device:C_Small
- added unit 6 of U101
- U101: footprint Package_DIP:DIP-14_W7.62mm -> Package_DIP:DIP-14_W7.62mm_Socket
- renumbered C101 to C102
Connections:
- net GND: now also C101.2, U101.12
- net VCC: now also C101.1, U101.13
Changed lines of the file:
@@
 	5700 4150 6000 4150
 $Comp
-L Device:C C101
+L Device:C C102
 U 1 1 5DA94A17
 P 5000 3600
-F 0 "C101" H 5115 3646 50  0000 L CNN
+F 0 "C102" H 5115 3646 50  0000 L CNN
 F 1 "4700pF" H 5115 3555 50  0000 L CNN
 F 2 "Capacitor_THT:C_Disc_D5.0mm_W2.5mm_P2.50mm" H 5038 3450 50  0001 C CNN
@@
 F 0 "U101" H 8130 3646 50  0000 L CNN
 F 1 "74AHCT04" H 8130 3555 50  0000 L CNN
-F 2 "Package_DIP:DIP-14_W7.62mm" H 7900 3600 50  0001 C CNN
+F 2 "Package_DIP:DIP-14_W7.62mm_Socket" H 7900 3600 50  0001 C CNN
 F 3 "https://assets.nexperia.com/documents/data-sheet/74HC_HCT04.pdf" H 7900 3600 50  0001 C CNN
 	7    7900 3600
@@
 	1    0    0    -1
 $EndComp
+$Comp
+L Device:C_Small C?
+U 1 1 5DA69FAE
+P 8350 3150
+AR Path="/5D9AAACD/5DA69FAE" Ref="C?"  Part="1"
+AR Path="/5D9A779A/5DA69FAE" Ref="C101"  Part="1"
+F 0 "C101" H 8442 3196 50  0000 L CNN
+F 1 ".1uF" H 8442 3105 50  0000 L CNN
+F 2 "Capacitor_THT:C_Disc_D5.0mm_W2.5mm_P2.50mm" H 8350 3150 50  0001 C CNN
+F 3 "~" H 8350 3150 50  0001 C CNN
+	1    8350 3150
+	1    0    0    -1
+$EndComp
+$Comp
+L power:GND #PWR?
+U 1 1 5DA69FB4
+P 8350 3250
+AR Path="/5D9AAACD/5DA69FB4" Ref="#PWR?"  Part="1"
+AR Path="/5D9A779A/5DA69FB4" Ref="#PWR0146"  Part="1"
+F 0 "#PWR0146" H 8350 3000 50  0001 C CNN
+F 1 "GND" H 8355 3077 50  0000 C CNN
+F 2 "" H 8350 3250 50  0001 C CNN
+F 3 "" H 8350 3250 50  0001 C CNN
+	1    8350 3250
+	1    0    0    -1
+$EndComp
+$Comp
+L power:VCC #PWR0147
+U 1 1 5DA6A4F9
+P 8350 3050
+F 0 "#PWR0147" H 8350 2900 50  0001 C CNN
+F 1 "VCC" H 8367 3223 50  0000 C CNN
+F 2 "" H 8350 3050 50  0001 C CNN
+F 3 "" H 8350 3050 50  0001 C CNN
+	1    8350 3050
+	1    0    0    -1
+$EndComp
+$Comp
+L 74xx:74HC04 U101
+U 6 1 5DAB0653
+P 7950 4900
+F 0 "U101" H 7950 5217 50  0000 C CNN
+F 1 "74AHCT04" H 7950 5126 50  0000 C CNN
+F 2 "Package_DIP:DIP-14_W7.62mm" H 7950 4900 50  0001 C CNN
+F 3 "https://assets.nexperia.com/documents/data-sheet/74HC_HCT04.pdf" H 7950 4900 50  0001 C CNN
+	6    7950 4900
+	1    0    0    -1
+$EndComp
+$Comp
+L power:VCC #PWR0156
+U 1 1 5DAB147B
+P 7650 4900
+F 0 "#PWR0156" H 7650 4750 50  0001 C CNN
+F 1 "VCC" V 7668 5027 50  0000 L CNN
+F 2 "" H 7650 4900 50  0001 C CNN
+F 3 "" H 7650 4900 50  0001 C CNN
+	1    7650 4900
+	0    -1   -1   0
+$EndComp
+$Comp
+L power:GND #PWR0157
+U 1 1 5DAB1787
+P 8250 4900
+F 0 "#PWR0157" H 8250 4650 50  0001 C CNN
+F 1 "GND" V 8255 4772 50  0000 R CNN
+F 2 "" H 8250 4900 50  0001 C CNN
+F 3 "" H 8250 4900 50  0001 C CNN
+	1    8250 4900
+	0    -1   -1   0
+$EndComp
 $EndSCHEMATC
