File: Power_Supplies/KWard_Adjustable_Bench_Power_Supply/design-files/pass-tube-array/pass-tube-array.kicad_pcb (KiCad board)
At the start: 2 copper layers, 130.8 x 142.9 mm, 26 parts, among them J1 Screw_Terminal_01x04, J2 Screw_Terminal_01x02, U1 6550, U2 6550, U3 6550, U4 6550

Commit message: Correct minor flaw in PCB.
Parts:
- moved J2 93.3 mm to (155.6, 159.4)
- moved REF** 93.3 mm to (91.4, 159.4)
- moved REF** 93.3 mm to (153.0, 76.8)
- moved U1 93.3 mm to (114.9, 66.7)
- moved U4 93.3 mm to (114.9, 135.3)
- moved J1 93.3 mm to (151.8, 25.4)
- moved R1 93.3 mm to (107.3, 39.4)
- moved R10 93.3 mm to (107.3, 104.8)
- moved R11 93.3 mm to (142.9, 123.8)
- moved R13 93.3 mm to (142.9, 144.1)
- moved R14 93.3 mm to (163.2, 144.1)
- moved R3 93.3 mm to (126.4, 39.4)
- moved R4 93.3 mm to (179.7, 39.4)
- moved R8 93.3 mm to (163.2, 123.8)
- moved REF** 93.3 mm to (91.4, 25.4)
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Routing:
- net Net-(J1-Pad3): track 190.1 -> 187.5 mm
